File: electrical/adapter1/adapter1/adapter1.kicad_pcb (KiCad board)
At the start: 2 copper layers, 12 x 49 mm, 5 parts, among them J2 Conn_01x08_Pin

Commit message: fix warnings
Parts:
- added TP1: TestPoint, TestPoint:TestPoint_Pad_1.5x1.5mm, F.Cu at (130.2, 80.2)
- added TP2: TestPoint, TestPoint:TestPoint_Pad_1.5x1.5mm, B.Cu at (130.2, 80.2)
- turned R1 to 180 degrees
Routing:
- net GND: track 174.6 -> 108.7 mm
- net /SLEEP: track 32.7 -> 40.1 mm
- net Net-(J1-BOARD_ID): track 32.9 -> 34.0 mm, vias 0 -> 2
- net /USB_P: vias 1 -> 0
- added copper zone on B.Cu, net +3V3
- added copper zone on B.Cu, net +5V
- added copper zone on F.Cu, net GND
Other:
- board text added: "+3V3"
- board text added: "nSLEEP"
