File: electrical/adapter1/adapter1/adapter1.kicad_pcb (KiCad board)
At the start: 2 copper layers, 12 x 49 mm, 7 parts, among them J2 Conn_01x08_Pin

Commit message: add silk text for stiffener
Other:
- board text added: "JLCJLCJLCJLC"
- board text added: "add stiffener and goldfingers here, please"
Changed lines of the file:
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@@
         (effects (font (size 1 1) (thickness 0.15)) (justify mirror))
+    )
+    (fp_text user "Diameter of pogo pins is 0.8mm." (at -8.5 6.5 unlocked) (layer "User.9")
+        (effects (font (size 1 1) (thickness 0.15)) (justify left bottom))
     )
     (fp_text user "but actual pogo pins seem more like 3.5mm." (at -8.5 8.25 unlocked) (layer "User.9")
@@
         (effects (font (size 1 1) (thickness 0.15)) (justify left bottom))
     )
-    (fp_text user "Diameter of pogo pins is 0.8mm." (at -8.5 6.5 unlocked) (layer "User.9")
-        (effects (font (size 1 1) (thickness 0.15)) (justify left bottom))
-    )
+    (fp_line (start -4.55 -3.4) (end -4.55 3.4)
+      (stroke (width 0.05) (type solid)) (layer "B.CrtYd"))
+    (fp_line (start -4.55 3.4) (end 4.55 3.4)
+      (stroke (width 0.05) (type solid)) (layer "B.CrtYd"))
+    (fp_line (start 4.55 -3.4) (end -4.55 -3.4)
+      (stroke (width 0.05) (type solid)) (layer "B.CrtYd"))
+    (fp_line (start 4.55 3.4) (end 4.55 -3.4)
+      (stroke (width 0.05) (type solid)) (layer "B.CrtYd"))
     (fp_line (start -5.25 -5.25) (end -5.25 5.25)
-      (stroke (width 0.12) (type solid)) (layer "B.SilkS"))
+      (stroke (width 0.12) (type solid)) (layer "User.8"))
     (fp_line (start -5.25 5.25) (end 5.25 5.25)
-      (stroke (width 0.12) (type solid)) (layer "B.SilkS"))
+      (stroke (width 0.12) (type solid)) (layer "User.8"))
     (fp_line (start 4.25 -5.25) (end -5.25 -5.25)
-      (stroke (width 0.12) (type solid)) (layer "B.SilkS"))
+      (stroke (width 0.12) (type solid)) (layer "User.8"))
     (fp_line (start 4.25 -5.25) (end 5.25 -4.25)
-      (stroke (width 0.12) (type solid)) (layer "B.SilkS"))
+      (stroke (width 0.12) (type solid)) (layer "User.8"))
     (fp_line (start 5.25 5.25) (end 5.25 -4.25)
-      (stroke (width 0.12) (type solid)) (layer "B.SilkS"))
-    (fp_line (start -4.55 -3.4) (end -4.55 3.4)
-      (stroke (width 0.05) (type solid)) (layer "B.CrtYd"))
-    (fp_line (start -4.55 3.4) (end 4.55 3.4)
-      (stroke (width 0.05) (type solid)) (layer "B.CrtYd"))
-    (fp_line (start 4.55 -3.4) (end -4.55 -3.4)
-      (stroke (width 0.05) (type solid)) (layer "B.CrtYd"))
-    (fp_line (start 4.55 3.4) (end 4.55 -3.4)
-      (stroke (width 0.05) (type solid)) (layer "B.CrtYd"))
+      (stroke (width 0.12) (type solid)) (layer "User.8"))
     (pad "1" thru_hole rect (at 3 -1.75 180) (size 1.6 2) (drill 0.6) (property pad_prop_testpoint) (layers "*.Cu" "B.Mask")
       (net 1 "GND") (pinfunction "GND") (pintype "input"))
@@
       (net 1 "GND") (pinfunction "Pin_8") (pintype "passive") (thermal_bridge_angle 45))
   )
+  (gr_line (start 123.25 82.25) (end 127.75 82.25)
+    (stroke (width 0.1) (type default)) (layer "F.SilkS"))
+  (gr_line (start 123.25 83) (end 127.75 87.5)
+    (stroke (width 0.1) (type default)) (layer "F.SilkS"))
+  (gr_line (start 123.25 86.75) (end 126 89.5)
+    (stroke (width 0.1) (type default)) (layer "F.SilkS"))
+  (gr_line (start 123.25 82.25) (end 127.75 86.75)
+    (stroke (width 0.1) (type default)) (layer "F.SilkS"))
+  (gr_line (start 124.75 82.25) (end 127.75 85.25)
+    (stroke (width 0.1) (type default)) (layer "F.SilkS"))
+  (gr_line (start 122.75 87) (end 122.75 86.25)
+    (stroke (width 0.1) (type default)) (layer "F.SilkS"))
+  (gr_line (start 126.25 82.25) (end 127.75 83.75)
+    (stroke (width 0.1) (type default)) (layer "F.SilkS"))
+  (gr_line (start 122.75 86.25) (end 122 86.25)
+    (stroke (width 0.1) (type default)) (layer "F.SilkS"))
+  (gr_line (start 123.25 89) (end 123.75 89.5)
+    (stroke (width 0.1) (type default)) (layer "F.SilkS"))
+  (gr_line (start 124 82.25) (end 127.75 86)
+    (stroke (width 0.1) (type default)) (layer "F.SilkS"))
+  (gr_line (start 122.75 86.25) (end 122.75 87)
+    (stroke (width 0.1) (type default)) (layer "F.SilkS"))
+  (gr_line (start 123.25 86) (end 126.75 89.5)
+    (stroke (width 0.1) (type default)) (layer "F.SilkS"))
+  (gr_line (start 127 82.25) (end 127.75 83)
+    (stroke (width 0.1) (type default)) (layer "F.SilkS"))
+  (gr_line (start 118.75 90) (end 122.75 86.25)
+    (stroke (width 0.1) (type default)) (layer "F.SilkS"))
+  (gr_line (start 125.5 82.25) (end 127.75 84.5)
+    (stroke (width 0.1) (type default)) (layer "F.SilkS"))
+  (gr_line (start 123.25 84.5) (end 127.75 89)
+    (stroke (width 0.1) (type default)) (layer "F.SilkS"))
+  (gr_line (start 123.25 87.5) (end 125.25 89.5)
+    (stroke (width 0.1) (type default)) (layer "F.SilkS"))
+  (gr_line (start 123.25 85.25) (end 127.5 89.5)
+    (stroke (width 0.1) (type default)) (layer "F.SilkS"))
+  (gr_line (start 123.25 83.75) (end 127.75 88.25)
+    (stroke (width 0.1) (type default)) (layer "F.SilkS"))
+  (gr_line (start 123.25 88.25) (end 124.5 89.5)
+    (stroke (width 0.1) (type default)) (layer "F.SilkS"))
   (gr_line (start 130.5 50.5) (end 130.5 40.5)
     (stroke (width 0.05) (type default)) (layer "Edge.Cuts"))
@@
     (effects (font (size 1 1) (thickness 0.2) bold) (justify left bottom mirror))
   )
+  (gr_text "JLCJLCJLCJLC" (at 121.25 61 90) (layer "B.SilkS")
+    (effects (font (size 1 1) (thickness 0.2) bold) (justify left bottom mirror))
+  )
   (gr_text "RUN" (at 125.75 76.25) (layer "F.SilkS")
     (effects (font (size 1 1) (thickness 0.2) bold) (justify left bottom))
@@
     (effects (font (size 1 1) (thickness 0.2)) (justify left bottom))
   )
+  (gr_text "add stiffener and\ngoldfingers here, please" (at 116.5 93.5) (layer "F.SilkS")
+    (effects (font (size 1 1) (thickness 0.1)) (justify left bottom))
+  )
   (gr_text "nSLEEP" (at 131.2 79.3 90) (layer "F.SilkS")
